File: _autosave-bilberry.kicad_pcb (KiCad board)
At the start: 4 copper layers, 85 x 56 mm, 173 parts, among them J1 Micro_SD_Card, J10 RF, J2 Conn_02x20_Odd_Even, J3 RJ45_LED_Shielded, J4 Conn_01x15_Male, J5 USB_OTG, J6 USB2, J7 USB2, J8 Conn_01x40_Male, J9 AudioJack4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

Commit message: update
Parts:
- moved R42 6.95 mm to (61.0, 45.4)
- moved C23 3.00 mm to (60.9, 42.2)
- moved C62 3.00 mm to (61.0, 38.9)
- moved L5 3.00 mm to (61.0, 40.5)
- moved R41 2.46 mm to (61.5, 42.5)
Routing:
- net EPHY-TXN: track 5.45 -> 6.12 mm
Changed lines of the file:
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@@
     (thickness 1.6)
     (drawings 26)
-    (tracks 279)
+    (tracks 281)
     (zones 0)
     (modules 173)
@@
   )
   (module Inductor_SMD:L_0603_1608Metric (layer F.Cu)
-    (at 60.95 43.46 180)
+    (at 60.95 40.46 180)
     (descr "Inductor SMD 0603 (1608 Metric), square (rectangular) end terminal, IPC_7351 nominal, (Body size source: http://www.tortai-tech.com/upload/download/2011102023233369053.pdf), generated with kicad-footprint-generator")
     (tags inductor)
@@
   )
   (module Capacitor_SMD:C_0603_1608Metric (layer F.Cu)
-    (at 60.95 41.85)
+    (at 60.95 38.85)
     (descr "Capacitor SMD 0603 (1608 Metric), square (rectangular) end terminal, IPC_7351 nominal, (Body size source: http://www.tortai-tech.com/upload/download/2011102023233369053.pdf), generated with kicad-footprint-generator")
     (tags capacitor)
@@
   )
   (module Capacitor_SMD:C_0603_1608Metric (layer F.Cu)
-    (at 60.94 45.17)
+    (at 60.94 42.17)
     (descr "Capacitor SMD 0603 (1608 Metric), square (rectangular) end terminal, IPC_7351 nominal, (Body size source: http://www.tortai-tech.com/upload/download/2011102023233369053.pdf), generated with kicad-footprint-generator")
     (tags capacitor)
@@
   )
   (module Resistor_SMD:R_0603_1608Metric (layer F.Cu)
-    (at 60.95 38.45)
+    (at 61.0375 45.4)
     (descr "Resistor SMD 0603 (1608 Metric), square (rectangular) end terminal, IPC_7351 nominal, (Body size source: http://www.tortai-tech.com/upload/download/2011102023233369053.pdf), generated with kicad-footprint-generator")
     (tags resistor)
@@
   )
   (module Resistor_SMD:R_0603_1608Metric (layer F.Cu)
-    (at 60.9625 40.15)
+    (at 61.5125 42.55)
     (descr "Resistor SMD 0603 (1608 Metric), square (rectangular) end terminal, IPC_7351 nominal, (Body size source: http://www.tortai-tech.com/upload/download/2011102023233369053.pdf), generated with kicad-footprint-generator")
     (tags resistor)
@@
   (segment (start 14.491 21.29) (end 13.506 22.275) (width 0.25) (layer F.Cu) (net 18))
   (segment (start 14.491 18.135) (end 14.491 21.29) (width 0.25) (layer F.Cu) (net 18))
-  (segment (start 63.7525 48.965) (end 61.7375 46.95) (width 0.25) (layer F.Cu) (net 30))
-  (segment (start 66.35 48.965) (end 63.7525 48.965) (width 0.25) (layer F.Cu) (net 30))
-  (segment (start 63.75 50.225) (end 68.89 50.225) (width 0.25) (layer F.Cu) (net 31))
-  (segment (start 62.175 48.65) (end 63.75 50.225) (width 0.25) (layer F.Cu) (net 31))
-  (segment (start 61.7375 48.65) (end 62.175 48.65) (width 0.25) (layer F.Cu) (net 31))
+  (segment (start 65.54 49.775) (end 66.35 48.965) (width 0.2) (layer F.Cu) (net 30))
+  (segment (start 64.5625 49.775) (end 65.54 49.775) (width 0.2) (layer F.Cu) (net 30))
+  (segment (start 61.7375 46.95) (end 64.5625 49.775) (width 0.2) (layer F.Cu) (net 30))
+  (segment (start 65.54 50.225) (end 68.89 50.225) (width 0.2) (layer F.Cu) (net 31))
+  (segment (start 64.376103 50.225) (end 65.54 50.225) (width 0.2) (layer F.Cu) (net 31))
+  (segment (start 62.801103 48.65) (end 64.376103 50.225) (width 0.2) (layer F.Cu) (net 31))
+  (segment (start 61.7375 48.65) (end 62.801103 48.65) (width 0.2) (layer F.Cu) (net 31))
   (segment (start 22.067 49.01) (end 19.5 46.443) (width 0.508) (layer F.Cu) (net 44))
   (segment (start 19.5 46.443) (end 19.5 45.45) (width 0.508) (layer F.Cu) (net 44))
