File: bilberry.kicad_pcb (KiCad board)
At the start: 4 copper layers, 85 x 56 mm, 173 parts, among them J1 Micro_SD_Card, J10 RF, J2 Conn_02x20_Odd_Even, J3 RJ45_LED_Shielded, J4 Conn_01x15_Male, J5 USB_OTG, J6 USB2, J7 USB2, J8 Conn_01x40_Male, J9 AudioJack4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

Commit message: update
Parts:
- moved R25 13.3 mm to (11.4, 7.02), turned to 0 degrees
- moved C29 7.06 mm to (14.5, 7.03), turned to 180 degrees
- moved L5 6.04 mm to (61.0, 40.5)
- moved R42 5.70 mm to (61.0, 45.4)
- moved C62 4.26 mm to (61.0, 38.9)
- moved C23 2.64 mm to (60.9, 42.2)
- moved R17 1.27 mm to (61.0, 47.0)
- moved R18 1.27 mm to (61.0, 48.6)
- moved R39 1.27 mm to (61.0, 36.8)
- moved R40 1.27 mm to (61.0, 35.2)
- moved R7 1.19 mm to (10.3, 39.6), turned to 0 degrees
- moved R41 1.19 mm to (61.5, 42.5)
- moved C7 0.31 mm to (10.3, 41.1), turned to 0 degrees
Connections:
- H1 pad 1: Net-(H1-Pad1) -> GND
- H2 pad 1: Net-(H2-Pad1) -> GND
- H3 pad 1: Net-(H3-Pad1) -> GND
- H4 pad 1: Net-(H4-Pad1) -> GND
- J8 pad 31: IO3V3 -> EPHY-VCC
- J8 pad 4: IO3V3 -> EPHY-VCC
- U4 pad 3: EPHY-VCC -> +5V
Routing:
- net GND: track 101.4 -> 185.6 mm, vias 2 -> 1
- net Net-(J3-Pad10): track 23.1 -> 0.00 mm
- net Net-(J3-Pad12): track 19.3 -> 0.00 mm
- net EPHY-RXP: track 16.4 -> 0.00 mm
- net EPHY-VCC: track 8.00 -> 23.2 mm
- net EPHY-RXN: track 14.1 -> 0.00 mm
- net ESP8089_XOUT: track 0.00 -> 12.1 mm
- net +5V: track 26.1 -> 38.2 mm
- net ESP8089_XIN: track 0.00 -> 11.8 mm
- net EPHY-RXM: track 11.8 -> 0.00 mm
- net EPHY-TXM: track 10.2 -> 0.00 mm
- net AVCC: track 0.00 -> 5.61 mm
- net IO3V3: track 0.00 -> 5.42 mm
- net Net-(C7-Pad2): track 11.7 -> 9.09 mm
- net WIFI_RESET: track 0.00 -> 2.37 mm
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Other:
- outline, holes or cut-outs redrawn
- rule trace_min: 0.2 -> 0.0635
