File: bilberry.sch (KiCad schematic (older format))
At the start: 174 parts, among them J1 Micro_SD_Card, J10 RF, J2 Conn_02x20_Odd_Even, J3 RJ45_LED_Shielded, J4 Conn_01x15_Male, J5 USB_OTG, J6 USB2, J7 USB2, J8 Conn_01x40_Male, J9 AudioJack4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

Commit message: update
Connections:
- net +3V3: now also J8.31 (Pin_31), J8.4 (Pin_4); no longer U4.3 (VIN)
- net +5V: now also U4.3 (VIN)
- net GND: now also H1.1, H2.1, H3.1, H4.1
- net IO3V3: no longer J8.31 (Pin_31), J8.4 (Pin_4)
Changed lines of the file:
@@
 	0    1    1    0
 $EndComp
-Text GLabel 17550 12050 0    50   Input ~ 0
-IO3V3
 Wire Wire Line
 	17550 11950 17650 11950
@@
 Text GLabel 17550 14650 0    50   Input ~ 0
 LCD_CLK
-Text GLabel 17550 14750 0    50   Input ~ 0
-IO3V3
 Text GLabel 17550 14850 0    50   Input ~ 0
 LCD_HSYNC
@@
 Connection ~ 4550 15950
 $Comp
-L power:+3V3 #PWR0124
-U 1 1 604E1F6B
-P 4450 15450
-F 0 "#PWR0124" H 4450 15300 50  0001 C CNN
-F 1 "+3V3" V 4465 15578 50  0000 L CNN
-F 2 "" H 4450 15450 50  0001 C CNN
-F 3 "" H 4450 15450 50  0001 C CNN
-	1    4450 15450
-	0    -1   -1   0
-$EndComp
-$Comp
 L Device:C C17
 U 1 1 5FD3DDC6
@@
 	0    -1   -1   0
 $EndComp
+$Comp
+L power:GND #PWR0172
+U 1 1 5F73C90F
+P 15800 8750
+F 0 "#PWR0172" H 15800 8500 50  0001 C CNN
+F 1 "GND" H 15805 8577 50  0000 C CNN
+F 2 "" H 15800 8750 50  0001 C CNN
+F 3 "" H 15800 8750 50  0001 C CNN
+	1    15800 8750
+	0    -1   -1   0
+$EndComp
+$Comp
+L power:GND #PWR0225
+U 1 1 5F73F618
+P 15800 9150
+F 0 "#PWR0225" H 15800 8900 50  0001 C CNN
+F 1 "GND" H 15805 8977 50  0000 C CNN
+F 2 "" H 15800 9150 50  0001 C CNN
+F 3 "" H 15800 9150 50  0001 C CNN
+	1    15800 9150
+	0    -1   -1   0
+$EndComp
+$Comp
+L power:GND #PWR0226
+U 1 1 5F73F90D
+P 15800 9550
+F 0 "#PWR0226" H 15800 9300 50  0001 C CNN
+F 1 "GND" H 15805 9377 50  0000 C CNN
+F 2 "" H 15800 9550 50  0001 C CNN
+F 3 "" H 15800 9550 50  0001 C CNN
+	1    15800 9550
+	0    -1   -1   0
+$EndComp
+$Comp
+L power:GND #PWR0227
+U 1 1 5F73FC20
+P 15800 9950
+F 0 "#PWR0227" H 15800 9700 50  0001 C CNN
+F 1 "GND" H 15805 9777 50  0000 C CNN
+F 2 "" H 15800 9950 50  0001 C CNN
+F 3 "" H 15800 9950 50  0001 C CNN
+	1    15800 9950
+	0    -1   -1   0
+$EndComp
+$Comp
+L power:+5V #PWR?
+U 1 1 5F7ABD74
+P 4450 15450
+F 0 "#PWR?" H 4450 15300 50  0001 C CNN
+F 1 "+5V" V 4465 15578 50  0000 L CNN
+F 2 "" H 4450 15450 50  0001 C CNN
+F 3 "" H 4450 15450 50  0001 C CNN
+	1    4450 15450
+	0    -1   -1   0
+$EndComp
+$Comp
+L power:+3V3 #PWR?
+U 1 1 5F84C8E9
+P 17550 12050
+F 0 "#PWR?" H 17550 11900 50  0001 C CNN
+F 1 "+3V3" V 17565 12178 50  0000 L CNN
+F 2 "" H 17550 12050 50  0001 C CNN
+F 3 "" H 17550 12050 50  0001 C CNN
+	1    17550 12050
+	0    -1   -1   0
+$EndComp
+$Comp
+L power:+3V3 #PWR?
+U 1 1 5F8EF300
+P 17550 14750
+F 0 "#PWR?" H 17550 14600 50  0001 C CNN
+F 1 "+3V3" V 17565 14878 50  0000 L CNN
+F 2 "" H 17550 14750 50  0001 C CNN
+F 3 "" H 17550 14750 50  0001 C CNN
+	1    17550 14750
+	0    -1   -1   0
+$EndComp
